Commit message: Typo fixed

File: description/robot_core.xacro (robot description, xacro)
@@ -34,10 +34,10 @@
             <material name="white"/>
         </visual>
-        <collission>
+        <collision>
             <origin xyz="0.15 0 0.075"/>
             <geometry>
                 <box size="0.3 0.3 0.15"/>
             </geometry>
-        </collission>
+        </collision>
         <xacro:inertial_box mass="0.5" x="0.3" y="0.3" z="0.15">
             <origin xyz="0.15 0 0.075" rpy="0 0 0"/>
@@ -58,10 +58,10 @@
             <material name="blue"/>
         </visual>
-        <collission>
+        <collision>
             <geometry>
                 <cylinder radius="0.05" length="0.04"/>
             </geometry>
-        </collission>
-        <xacro:inertial_cylinder mass="0.1" radius="0.05" length="0.4">
+        </collision>
+        <xacro:inertial_cylinder mass="0.1" radius="0.05" length="0.04">
             <origin xyz="0 0 0" rpy="0 0 0"/>
         </xacro:inertial_cylinder>
@@ -81,10 +81,10 @@
             <material name="blue"/>
         </visual>
-        <collission>
+        <collision>
             <geometry>
                 <cylinder radius="0.05" length="0.04"/>
             </geometry>
-        </collission>
-        <xacro:inertial_cylinder mass="0.1" radius="0.05" length="0.4">
+        </collision>
+        <xacro:inertial_cylinder mass="0.1" radius="0.05" length="0.04">
             <origin xyz="0 0 0" rpy="0 0 0"/>
         </xacro:inertial_cylinder>
@@ -103,9 +103,9 @@
             <material name="black"/>
         </visual>
-        <collission>
+        <collision>
             <geometry>
                 <sphere radius="0.05"/>
             </geometry>
-        </collission>
+        </collision>
         <xacro:inertial_sphere mass="0.1" radius="0.05">
             <origin xyz="0 0 0" rpy="0 0 0"/>

Commit message: Gazebo color added

File: description/robot_core.xacro (robot description, xacro)
@@ -44,4 +44,7 @@
         </xacro:inertial_box>
     </link>
+    <gazebo reference="chassis">
+        <material>Gazebo/White</material>
+    </gazebo>
     <!-- LEFT WHEEL JOINT -->
     <joint name="left_wheel_joint" type="continuous">
@@ -67,4 +70,7 @@
         </xacro:inertial_cylinder>
     </link>
+    <gazebo reference="left_wheel">
+        <material>Gazebo/Blue</material>
+    </gazebo>
     <!-- RIGHT WHEEL JOINT -->
     <joint name="right_wheel_joint" type="continuous">
@@ -90,4 +96,7 @@
         </xacro:inertial_cylinder>
     </link>
+    <gazebo reference="right_wheel">
+        <material>Gazebo/Blue</material>
+    </gazebo>
     <!-- CASTER WHEEL JOINT -->
     <joint name="caster_wheel_joint" type="fixed">
@@ -112,3 +121,6 @@
         </xacro:inertial_sphere>
     </link>
+    <gazebo reference="caster_wheel">
+        <material>Gazebo/Black</material>
+    </gazebo>
 </robot>
