Commit message: current version of the robot

File: description/gazebo_control.xacro (robot description, xacro)
@@ -6,6 +6,6 @@
         <left_joint>left_wheel_joint</left_joint>
         <right_joint>right_wheel_joint</right_joint>
-        <wheel_separation>0.35</wheel_separation>
-        <wheel_diameter>0.1</wheel_diameter>
+        <wheel_separation>0.185</wheel_separation>
+        <wheel_diameter>0.0678</wheel_diameter>
         <!-- Limits -->
         <max_wheel_torque>200</max_wheel_torque>

File: description/lidar.xacro (robot description, xacro)
@@ -2,11 +2,12 @@
 <robot xmlns:xacro="http://www.ros.org/wiki/xacro">
   <xacro:property name="laser_offset_x" value="0.115"/>
-  <xacro:property name="laser_offset_z" value="0.01"/>
+  <xacro:property name="laser_offset_z" value="0.002"/><!-- 0.2cm = 0.002-->
   <xacro:property name="laser_radius" value="0.035"/>
-  <xacro:property name="laser_thickness" value="0.055"/>
+  <xacro:property name="laser_thickness" value="0.02"/><!-- 3.5 + 1.2 + 0.8 -->
+  <xacro:property name="laser_base_height" value="0.035"/>
   <joint name="laser_joint" type="fixed">
     <parent link="chassis" />
     <child link="laser_frame" />
-    <origin xyz="${laser_offset_x} 0 ${chassis_height+laser_thickness/2}" rpy="0 0 0" />
+    <origin xyz="${laser_offset_x} 0 ${chassis_height+laser_base_height+laser_thickness/2}" rpy="0 0 0" />
   </joint>
   <link name="laser_frame">
@@ -16,5 +17,12 @@
         <cylinder radius="${laser_radius}" length="${laser_thickness}"/>
       </geometry>
-      <material name="red"/>
+      <material name="black"/>
+    </visual>
+    <visual>
+      <origin xyz="0 0 ${-laser_offset_z-laser_thickness/2-laser_base_height/2}" rpy="0 0 0" />
+      <geometry>
+        <cylinder radius="${0.005}" length="${laser_base_height}"/>
+      </geometry>
+      <material name="black"/>
     </visual>
     <collision>
@@ -23,5 +31,5 @@
       </geometry>
     </collision>
-    <xacro:inertial_cylinder mass="0.3" radius="${laser_radius}" length="${laser_thickness}">
+    <xacro:inertial_cylinder mass="0.2" radius="${laser_radius}" length="${laser_thickness}">
       <origin xyz="0 0 0" rpy="0 0 0"/>
     </xacro:inertial_cylinder>
@@ -50,5 +58,5 @@
       <plugin name="laser_controller" filename="libgazebo_ros_ray_sensor.so">
         <ros>
-          <argument>--ros-args --remap ~/out:=scan</argument>
+          <argument>~/out:=scan</argument>
         </ros>
         <output_type>sensor_msgs/LaserScan</output_type>

File: description/robot.urdf.xacro (robot description, xacro)
@@ -1,7 +1,13 @@
 <?xml version="1.0"?>
 <robot xmlns:xacro="http://www.ros.org/wiki/xacro" name="robot">
-    <xacro:include filename="robot_core.xacro"/>
-    <!-- <xacro:include filename="gazebo_control.xacro"/> -->
-    <xacro:include filename="ros2_control.xacro"/>
+    <xacro:arg name="use_ros2_control" default="true"/>
+    <xacro:arg name="sim_mode" default="false"/>
+    <xacro:include filename="robot_core.xacro" />
+    <xacro:if value="$(arg use_ros2_control)">
+        <xacro:include filename="ros2_control.xacro" />
+    </xacro:if>
+    <xacro:unless value="$(arg use_ros2_control)">
+        <xacro:include filename="gazebo_control.xacro" />
+    </xacro:unless>
     <xacro:include filename="lidar.xacro"/>
     <xacro:include filename="camera.xacro"/>

File: description/ros2_control.xacro (robot description, xacro)
@@ -1,28 +1,61 @@
 <?xml version="1.0"?>
 <robot xmlns:xacro="http://www.ros.org/wiki/xacro">
-    <ros2_control name="GazeboSystem" type="system">
-        <hardware>
-            <plugin>gazebo_ros2_control/GazeboSystem</plugin>
-        </hardware>
-        <joint name="left_wheel_joint">
-            <command_interface name="velocity">
-                <param name="min">-10</param>
-                <param name="max">10</param>
-            </command_interface>
-            <state_interface name="velocity"/>
-            <state_interface name="position"/>
-        </joint>
-        <joint name="right_wheel_joint">
-            <command_interface name="velocity">
-                <param name="min">-10</param>
-                <param name="max">10</param>
-            </command_interface>
-            <state_interface name="velocity"/>
-            <state_interface name="position"/>
-        </joint>
-    </ros2_control>
+    <xacro:unless value="$(arg sim_mode)">
+        <ros2_control name="RealRobot" type="system">
+            <hardware>
+                <plugin>diffdrive_arduino/DiffDriveArduino</plugin>
+                <param name="left_wheel_name">left_wheel_joint</param>
+                <param name="right_wheel_name">right_wheel_joint</param>
+                <param name="loop_rate">30</param>
+                <param name="device">/dev/ttyACM0</param>
+                <param name="baud_rate">57600</param>
+                <param name="timeout">1000</param>
+                <param name="enc_counts_per_rev">1400</param>
+            </hardware>
+            <joint name="left_wheel_joint">
+                <command_interface name="velocity">
+                    <param name="min">-10</param>
+                    <param name="max">10</param>
+                </command_interface>
+                <state_interface name="velocity"/>
+                <state_interface name="position"/>
+            </joint>
+            <joint name="right_wheel_joint">
+                <command_interface name="velocity">
+                    <param name="min">-10</param>
+                    <param name="max">10</param>
+                </command_interface>
+                <state_interface name="velocity"/>
+                <state_interface name="position"/>
+            </joint>
+        </ros2_control>
+    </xacro:unless>
+    <xacro:if value="$(arg sim_mode)">
+        <ros2_control name="GazeboSystem" type="system">
+            <hardware>
+                <plugin>gazebo_ros2_control/GazeboSystem</plugin>
+            </hardware>
+            <joint name="left_wheel_joint">
+                <command_interface name="velocity">
+                    <param name="min">-10</param>
+                    <param name="max">10</param>
+                </command_interface>
+                <state_interface name="velocity"/>
+                <state_interface name="position"/>
+            </joint>
+            <joint name="right_wheel_joint">
+                <command_interface name="velocity">
+                    <param name="min">-10</param>
+                    <param name="max">10</param>
+                </command_interface>
+                <state_interface name="velocity"/>
+                <state_interface name="position"/>
+            </joint>
+        </ros2_control>
+    </xacro:if>
     <gazebo>
         <plugin name="gazebo_ros2_control" filename="libgazebo_ros2_control.so">
             <parameters>$(find ks-robo-car)/config/car_controllers.yaml</parameters>
+            <parameters>$(find ks-robo-car)/config/gaz_ros2_ctl_use_sim.yaml</parameters>
         </plugin>
     </gazebo>
