Commit message: URDF updated with actual dimensions

File: description/camera.xacro (robot description, xacro)
@@ -1,13 +1,16 @@
 <?xml version="1.0"?>
 <robot xmlns:xacro="http://www.ros.org/wiki/xacro" >
+    <xacro:property name="camera_length" value="0.001"/>
+    <xacro:property name="camera_width" value="0.020"/>
+    <xacro:property name="camera_height" value="0.025"/>
     <joint name="camera_joint" type="fixed">
         <parent link="chassis"/>
         <child link="camera_link"/>
-        <origin xyz="0.305 0 0.08" rpy="0 0 0"/>
+        <origin xyz="${chassis_length+camera_length} 0 ${chassis_height/2}" rpy="0 0 0"/>
     </joint>
     <link name="camera_link">
         <visual>
             <geometry>
-                <box size="0.010 0.03 0.03"/>
+                <box size="${camera_length} ${camera_width} ${camera_height}"/>
             </geometry>
             <material name="red"/>

File: description/lidar.xacro (robot description, xacro)
@@ -1,13 +1,18 @@
 <?xml version="1.0"?>
 <robot xmlns:xacro="http://www.ros.org/wiki/xacro">
+  <xacro:property name="laser_offset_x" value="0.115"/>
+  <xacro:property name="laser_offset_z" value="0.01"/>
+  <xacro:property name="laser_radius" value="0.035"/>
+  <xacro:property name="laser_thickness" value="0.055"/>
   <joint name="laser_joint" type="fixed">
     <parent link="chassis" />
     <child link="laser_frame" />
-    <origin xyz="0.1 0 0.175" rpy="0 0 0" />
+    <origin xyz="${laser_offset_x} 0 ${chassis_height+laser_thickness/2}" rpy="0 0 0" />
   </joint>
   <link name="laser_frame">
     <visual>
+      <origin xyz="0 0 ${-laser_offset_z}" rpy="0 0 0" />
       <geometry>
-        <cylinder radius="0.05" length="0.04"/>
+        <cylinder radius="${laser_radius}" length="${laser_thickness}"/>
       </geometry>
       <material name="red"/>
@@ -15,8 +20,8 @@
     <collision>
       <geometry>
-        <cylinder radius="0.05" length="0.04"/>
+        <cylinder radius="${laser_radius}" length="${laser_thickness}"/>
       </geometry>
     </collision>
-    <xacro:inertial_cylinder mass="0.1" radius="0.05" length="0.04">
+    <xacro:inertial_cylinder mass="0.3" radius="${laser_radius}" length="${laser_thickness}">
       <origin xyz="0 0 0" rpy="0 0 0"/>
     </xacro:inertial_cylinder>

File: description/robot_core.xacro (robot description, xacro)
@@ -2,4 +2,18 @@
 <robot xmlns:xacro="http://www.ros.org/wiki/xacro">
     <xacro:include filename="inertial_macros.xacro"/>
+    <xacro:property name="chassis_length" value="0.255"/>
+    <xacro:property name="chassis_width" value="0.15"/>
+    <xacro:property name="chassis_height" value="0.034"/>
+    <xacro:property name="chassis_mass" value="1.0"/>
+    <xacro:property name="wheel_radius" value="0.0339"/>
+    <xacro:property name="wheel_thickness" value="0.025"/>
+    <xacro:property name="wheel_mass" value="0.05"/>
+    <xacro:property name="wheel_offset_x" value="0.07"/>
+    <xacro:property name="wheel_offset_y" value="0.0925"/>
+    <xacro:property name="wheel_offset_z" value="0.0031"/>
+    <xacro:property name="caster_wheel_radius" value="0.01"/>
+    <xacro:property name="caster_wheel_mass" value="0.01"/>
+    <xacro:property name="caster_wheel_offset_x" value="0.19"/>
+    <xacro:property name="caster_wheel_offset_z" value="${wheel_offset_z + wheel_radius - caster_wheel_radius}"/>
     <material name="white">
         <color rgba="1 1 1 1" />
@@ -20,30 +34,38 @@
     <link name="base_link">
     </link>
+    <!-- BASE_FOOTPRINT LINK -->
+    <joint name="base_footprint_joint" type="fixed">
+        <parent link="base_link"/>
+        <child link="base_footprint"/>
+        <origin xyz="0 0 0" rpy="0 0 0"/>
+    </joint>
+    <link name="base_footprint">
+    </link>
     <!-- CHASSIS LINK -->
     <joint name="chassis_joint" type="fixed">
         <parent link="base_link"/>
         <child link="chassis"/>
-        <origin xyz="-0.1 0 0"/> <!-- Child frame w.r.t. parent frame -->
+        <origin xyz="${-wheel_offset_x} 0 ${wheel_offset_z}"/>
     </joint>
     <link name="chassis">
         <visual>
-            <origin xyz="0.15 0 0.075"/>
+            <origin xyz="${chassis_length/2} 0 ${chassis_height/2}"/>
             <geometry>
-                <box size="0.3 0.3 0.15"/>
+                <box size="${chassis_length} ${chassis_width} ${chassis_height}"/>
             </geometry>
-            <material name="white"/>
+            <material name="orange"/>
         </visual>
         <collision>
-            <origin xyz="0.15 0 0.075"/>
+            <origin xyz="${chassis_length/2} 0 ${chassis_height/2}"/>
             <geometry>
-                <box size="0.3 0.3 0.15"/>
+                <box size="${chassis_length} ${chassis_width} ${chassis_height}"/>
             </geometry>
         </collision>
-        <xacro:inertial_box mass="0.5" x="0.3" y="0.3" z="0.15">
-            <origin xyz="0.15 0 0.075" rpy="0 0 0"/>
+        <xacro:inertial_box mass="0.5" x="${chassis_length}" y="${chassis_width}" z="${chassis_height}">
+            <origin xyz="${chassis_length/2} 0 ${chassis_height/2}" rpy="0 0 0"/>
         </xacro:inertial_box>
     </link>
     <gazebo reference="chassis">
-        <material>Gazebo/White</material>
+        <material>Gazebo/Orange</material>
     </gazebo>
     <!-- LEFT WHEEL JOINT -->
@@ -51,11 +73,11 @@
         <parent link="base_link"/>
         <child link="left_wheel"/>
-        <origin xyz="0 0.175 0" rpy="-${pi/2} 0 0"/> <!-- Child frame w.r.t. parent frame -->
-        <axis xyz="0 0 1" />
+        <origin xyz="0 ${wheel_offset_y} 0" rpy="-${pi/2} 0 0" />
+        <axis xyz="0 0 1"/>
     </joint>
     <link name="left_wheel">
         <visual>
             <geometry>
-                <cylinder radius="0.05" length="0.04"/>
+                <cylinder radius="${wheel_radius}" length="${wheel_thickness}"/>
             </geometry>
             <material name="blue"/>
@@ -63,8 +85,8 @@
         <collision>
             <geometry>
-                <cylinder radius="0.05" length="0.04"/>
+                <sphere radius="${wheel_radius}"/>
             </geometry>
         </collision>
-        <xacro:inertial_cylinder mass="0.1" radius="0.05" length="0.04">
+        <xacro:inertial_cylinder mass="${wheel_mass}" length="${wheel_thickness}" radius="${wheel_radius}">
             <origin xyz="0 0 0" rpy="0 0 0"/>
         </xacro:inertial_cylinder>
@@ -77,11 +99,11 @@
         <parent link="base_link"/>
         <child link="right_wheel"/>
-        <origin xyz="0 -0.175 0" rpy="${pi/2} 0 0"/> <!-- Child frame w.r.t. parent frame -->
-        <axis xyz="0 0 -1" />
+        <origin xyz="0 ${-wheel_offset_y} 0" rpy="${pi/2} 0 0" />
+        <axis xyz="0 0 -1"/>
     </joint>
     <link name="right_wheel">
         <visual>
             <geometry>
-                <cylinder radius="0.05" length="0.04"/>
+                <cylinder radius="${wheel_radius}" length="${wheel_thickness}"/>
             </geometry>
             <material name="blue"/>
@@ -89,8 +111,8 @@
         <collision>
             <geometry>
-                <cylinder radius="0.05" length="0.04"/>
+                <sphere radius="${wheel_radius}"/>
             </geometry>
         </collision>
-        <xacro:inertial_cylinder mass="0.1" radius="0.05" length="0.04">
+        <xacro:inertial_cylinder mass="${wheel_mass}" length="${wheel_thickness}" radius="${wheel_radius}">
             <origin xyz="0 0 0" rpy="0 0 0"/>
         </xacro:inertial_cylinder>
@@ -100,30 +122,50 @@
     </gazebo>
     <!-- CASTER WHEEL JOINT -->
+    <joint name="caster_wheel_base_joint" type="fixed">
+        <parent link="chassis"/>
+        <child link="caster_wheel_base"/>
+        <origin xyz="${caster_wheel_offset_x} 0 ${-caster_wheel_offset_z/2}"/>
+    </joint>
+    <link name="caster_wheel_base">
+        <visual>
+            <geometry>
+                <box size="${caster_wheel_radius*2} ${caster_wheel_radius*2} ${caster_wheel_offset_z}"/>
+            </geometry>
+            <material name="white"/>
+        </visual>
+        <collision>
+            <geometry>
+                <box size="${caster_wheel_radius*2} ${caster_wheel_radius*2} ${caster_wheel_offset_z}"/>
+            </geometry>
+        </collision>
+        <xacro:inertial_box mass="0.01" x="${caster_wheel_radius*2}" y="${caster_wheel_radius*2}" z="${caster_wheel_offset_z}">
+            <origin xyz="${caster_wheel_radius/2} 0 ${caster_wheel_offset_z/2}" rpy="0 0 0"/>
+        </xacro:inertial_box>
+    </link>
     <joint name="caster_wheel_joint" type="fixed">
-        <parent link="chassis" />
-        <child link="caster_wheel" />
-        <origin xyz="0.24 0 0" /> <!-- Child frame w.r.t. parent frame -->
+        <parent link="chassis"/>
+        <child link="caster_wheel"/>
+        <origin xyz="${caster_wheel_offset_x} 0 ${-caster_wheel_offset_z}"/>
     </joint>
     <link name="caster_wheel">
         <visual>
             <geometry>
-                <sphere radius="0.05"/>
+                <sphere radius="${caster_wheel_radius}"/>
             </geometry>
-            <material name="black"/>
+            <material name="white"/>
         </visual>
         <collision>
             <geometry>
-                <sphere radius="0.05"/>
+                <sphere radius="${caster_wheel_radius}"/>
             </geometry>
         </collision>
-        <xacro:inertial_sphere mass="0.1" radius="0.05">
+        <xacro:inertial_sphere mass="${caster_wheel_mass}" radius="${caster_wheel_radius}">
             <origin xyz="0 0 0" rpy="0 0 0"/>
         </xacro:inertial_sphere>
     </link>
     <gazebo reference="caster_wheel">
-        <material>Gazebo/Black</material>
-        <!-- Making it frictionless in Gazebo -->
-        <mu1 value="0.001" />
-        <mu2 value="0.001" />
+        <material>Gazebo/White</material>
+        <mu1 value="0.001"/>
+        <mu2 value="0.001"/>
     </gazebo>
 </robot>

Commit message: dev machine extra files

File: description/camera.xacro (robot description, xacro)
@@ -7,5 +7,5 @@
         <parent link="chassis"/>
         <child link="camera_link"/>
-        <origin xyz="${chassis_length+camera_length} 0 ${chassis_height/2}" rpy="0 0 0"/>
+        <origin xyz="${chassis_length+camera_length} 0 ${chassis_height/2}" rpy="0 0.18 0"/>
     </joint>
     <link name="camera_link">
